Commit message: add lidar

File: simple_bot_ws/src/simple_bot/description/robot_2wd.urdf (robot description, URDF)
Before this commit: robot robot, 5 links, 4 joints
Links:
- added link laser_frame, mass 0.1; collision cylinder length=0.04 radius=0.05; visual cylinder length=0.04 radius=0.05
Joints:
- added joint laser_joint: type fixed, parent chassis, child laser_frame, origin xyz=0.1 0 0.175 rpy=0 0 0

Commit message: camera added

File: simple_bot_ws/src/simple_bot/description/robot_2wd.urdf (robot description, URDF)
Before this commit: robot robot, 6 links, 5 joints
Links:
- added link camera_link; visual box size=0.010 0.03 0.03
- added link camera_link_optical
Joints:
- added joint camera_joint: type fixed, parent chassis, child camera_link, origin xyz=0.305 0 0.08 rpy=0 0 0
- added joint camera_optical_joint: type fixed, parent camera_link, child camera_link_optical, origin xyz=0 0 0 rpy=-1.57 0 -1.57
